File: pcb/Lily58.kicad_pcb (KiCad board)
At the start: 2 copper layers, 142.5 x 106.3 mm, 116 parts, among them J1 LED, P4 OLED, SW1 SW_PUSH, SW10 SW_PUSH, SW11 SW_PUSH, SW12 SW_PUSH, SW13 SW_PUSH, SW14 SW_PUSH, SW15 SW_PUSH, SW16 SW_PUSH, SW17 SW_PUSH, SW18 SW_PUSH, SW19 SW_PUSH, SW2 SW_PUSH, SW20 SW_PUSH, SW21 SW_PUSH, SW22 SW_PUSH, SW23 SW_PUSH, SW24 SW_PUSH, SW25 Rotary_Encoder_Switch, SW26 SW_PUSH, SW27 SW_PUSH, SW28 SW_PUSH, SW29 SW_PUSH, SW3 SW_PUSH, SW4 SW_PUSH, SW5 SW_PUSH, SW6 SW_PUSH, SW7 SW_PUSH, SW8 SW_PUSH, SW9 SW_PUSH, U1 NiceNano

Commit message: Some more wiring updates
Parts:
- removed J1: LED, Lily58-footprint:StripLED
- added J+1: Conn_01x01_Male, TestPoint:TestPoint_Pad_2.0x2.0mm, F.Cu at (86.1, 71.1)
- added J-1: Conn_01x01_Male, TestPoint:TestPoint_Pad_2.0x2.0mm, F.Cu at (86.1, 67.1)
Connections:
- L10 pad 4: VCC -> Net-(D_LED1-Pad1)
- L11 pad 4: VCC -> Net-(D_LED1-Pad1)
- L12 pad 4: VCC -> Net-(D_LED1-Pad1)
- L13 pad 4: VCC -> Net-(D_LED1-Pad1)
- L14 pad 4: VCC -> Net-(D_LED1-Pad1)
- L15 pad 4: VCC -> Net-(D_LED1-Pad1)
- L16 pad 4: VCC -> Net-(D_LED1-Pad1)
- L17 pad 4: VCC -> Net-(D_LED1-Pad1)
- L18 pad 4: VCC -> Net-(D_LED1-Pad1)
- L19 pad 4: VCC -> Net-(D_LED1-Pad1)
- L20 pad 4: VCC -> Net-(D_LED1-Pad1)
- L21 pad 4: VCC -> Net-(D_LED1-Pad1)
- L22 pad 4: VCC -> Net-(D_LED1-Pad1)
- L23 pad 4: VCC -> Net-(D_LED1-Pad1)
- L24 pad 4: VCC -> Net-(D_LED1-Pad1)
- L25 pad 4: VCC -> Net-(D_LED1-Pad1)
- L26 pad 4: VCC -> Net-(D_LED1-Pad1)
- L27 pad 4: VCC -> Net-(D_LED1-Pad1)
- L28 pad 4: VCC -> Net-(D_LED1-Pad1)
- L29 pad 4: VCC -> Net-(D_LED1-Pad1)
- L30 pad 4: VCC -> Net-(D_LED1-Pad1)
- L34 pad 4: VCC -> unconnected-(D_LED1-Pad2)
- L35 pad 4: VCC -> unconnected-(D_LED1-Pad2)
- L36 pad 4: VCC -> unconnected-(D_LED1-Pad2)
- L7 pad 4: VCC -> Net-(D_LED1-Pad1)
- L8 pad 4: VCC -> Net-(D_LED1-Pad1)
- L9 pad 4: VCC -> Net-(D_LED1-Pad1)
- SW_Battery1 pad 2: unconnected-(SW_Battery1-Pad2) -> Net-(SW_Battery1-Pad2)
Routing:
- net Net-(D_LED1-Pad1): track 11.4 -> 801.3 mm, vias 0 -> 33
- net GND: track 311.1 -> 686.4 mm, vias 8 -> 19
- net unconnected-(D_LED1-Pad2): track 5.83 -> 310.7 mm, vias 0 -> 16
- net col2: track 63.3 -> 261.4 mm, vias 3 -> 14
- net row0: track 91.0 -> 237.0 mm, vias 2 -> 10
- net col1: track 193.3 -> 323.3 mm, vias 7 -> 12
- net row1: track 26.7 -> 140.3 mm, vias 1 -> 4
- net SDA: track 133.2 -> 32.3 mm, vias 16 -> 7
- net col3: track 176.2 -> 261.7 mm, vias 7 -> 8
- net LED: track 67.7 -> 0.00 mm, vias 4 -> 0
- net col5: track 76.0 -> 138.1 mm, vias 2 -> 5
- net row3: track 87.5 -> 141.1 mm, vias 0 -> 2
- net col4: track 190.6 -> 241.3 mm, vias 7 -> 8
- net row2: track 82.5 -> 132.7 mm
- net Net-(SW_Battery1-Pad2): track 0.00 -> 48.1 mm, vias 0 -> 2
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